File: KiCad/HeatPumpControl.kicad_sch (KiCad schematic)
At the start: 46 parts, among them J1 Conn_01x04_Male, J2 Conn_01x04_Male, J3 Conn_01x04_Male, J4 Conn_01x03_Male, Q1 2N2222A, Q2 Q_PMOS_GDS, U1 TSOP23xx, U3 XIAO-ESP32-C6-SMD

Commit message: DRC changes
Parts:
- D3, D6: value ~ -> (none)
